File: eagleproject.sch (EAGLE design)
At the start: 0 parts

Commit message: sparkfun libraries i didn't have
Parts:
- added C1: 0.1uF, SparkFun-Capacitors:0.1UF-0603-25V-(+80/-20%)
- added J1: RASPBERRYPI-40-PIN-GPIO_PTH, SparkFun-Connectors:RASPBERRYPI-40-PIN-GPIO_PTH
- added R1: 100, SparkFun-Resistors:100OHM-0603-1/4W-5%
- added U$1: MAX485DIL, SparkFun-Retired:MAX485DIL
Connections:
- new net 5V: C1.1, J1.5V@2, J1.5V@4, U$1.VCC
- new net A: R1.2, U$1.A
- new net B: R1.1, U$1.B
- new net GND: C1.2, U$1.GND

Commit message: velleman user manual
Parts:
- added J2: XLR-3-FEMALE, SparkFun-Connectors:XLR-3-FEMALE
- added J3: XLR-3-MALE, SparkFun-Connectors:XLR-3-MALE
Connections:
- net A: now also J2.D+, J3.D+
- net B: now also J2.D-, J3.D-
- net GND: now also J1.GND@14, J1.GND@20, J1.GND@25, J1.GND@30, J1.GND@34, J1.GND@39, J1.GND@6, J1.GND@9, J2.GND, J3.GND
Changed lines of the file:
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@@
 <part name="SUPPLY3" library="SparkFun-PowerSymbols" library_urn="urn:adsk.eagle:library:530" deviceset="5V" device=""/>
 <part name="R1" library="SparkFun-Resistors" library_urn="urn:adsk.eagle:library:532" deviceset="100OHM" device="-0603-1/4W-5%" package3d_urn="urn:adsk.eagle:package:39650/1" value="100"/>
+<part name="J2" library="SparkFun-Connectors" deviceset="XLR-3" device="-FEMALE"/>
+<part name="J3" library="SparkFun-Connectors" deviceset="XLR-3" device="-MALE"/>
+<part name="GND3" library="SparkFun-PowerSymbols" library_urn="urn:adsk.eagle:library:530" deviceset="DGND" device=""/>
+<part name="GND4" library="SparkFun-PowerSymbols" library_urn="urn:adsk.eagle:library:530" deviceset="DGND" device=""/>
 </parts>
 <sheets>
@@
 <attribute name="VALUE" x="81.28" y="48.006" size="1.778" layer="96" align="top-center"/>
 </instance>
-<instance part="SUPPLY3" gate="G$1" x="5.08" y="96.52" smashed="yes">
-<attribute name="VALUE" x="5.08" y="99.314" size="1.778" layer="96" align="bottom-center"/>
+<instance part="SUPPLY3" gate="G$1" x="2.54" y="93.98" smashed="yes">
+<attribute name="VALUE" x="2.54" y="96.774" size="1.778" layer="96" align="bottom-center"/>
 </instance>
 <instance part="R1" gate="G$1" x="96.52" y="58.42" smashed="yes">
 <attribute name="NAME" x="96.52" y="59.944" size="1.778" layer="95" font="vector" align="bottom-center"/>
 <attribute name="VALUE" x="96.52" y="56.896" size="1.778" layer="96" font="vector" align="top-center"/>
+</instance>
+<instance part="J2" gate="G$1" x="81.28" y="111.76" smashed="yes">
+<attribute name="NAME" x="76.2" y="119.634" size="1.778" layer="95" font="vector"/>
+<attribute name="VALUE" x="76.2" y="101.6" size="1.778" layer="96" font="vector"/>
+</instance>
+<instance part="J3" gate="G$1" x="106.68" y="111.76" smashed="yes" rot="MR0">
+<attribute name="NAME" x="111.76" y="119.634" size="1.778" layer="95" font="vector" rot="MR0"/>
+<attribute name="VALUE" x="111.76" y="101.6" size="1.778" layer="96" font="vector" rot="MR0"/>
+</instance>
+<instance part="GND3" gate="G$1" x="93.98" y="96.52" smashed="yes">
+<attribute name="VALUE" x="93.98" y="96.266" size="1.778" layer="96" align="top-center"/>
+</instance>
+<instance part="GND4" gate="G$1" x="2.54" y="30.48" smashed="yes">
+<attribute name="VALUE" x="2.54" y="30.226" size="1.778" layer="96" align="top-center"/>
 </instance>
 </instances>
@@
 <segment>
 <pinref part="J1" gate="G$1" pin="5V@2"/>
-<wire x1="7.62" y1="91.44" x2="5.08" y2="91.44" width="0.1524" layer="91"/>
+<wire x1="7.62" y1="91.44" x2="2.54" y2="91.44" width="0.1524" layer="91"/>
 <pinref part="SUPPLY3" gate="G$1" pin="5V"/>
-<wire x1="5.08" y1="91.44" x2="5.08" y2="96.52" width="0.1524" layer="91"/>
+<wire x1="2.54" y1="91.44" x2="2.54" y2="93.98" width="0.1524" layer="91"/>
 <pinref part="J1" gate="G$1" pin="5V@4"/>
-<wire x1="7.62" y1="88.9" x2="5.08" y2="88.9" width="0.1524" layer="91"/>
-<wire x1="5.08" y1="88.9" x2="5.08" y2="91.44" width="0.1524" layer="91"/>
-<junction x="5.08" y="91.44"/>
+<wire x1="7.62" y1="88.9" x2="2.54" y2="88.9" width="0.1524" layer="91"/>
+<wire x1="2.54" y1="88.9" x2="2.54" y2="91.44" width="0.1524" layer="91"/>
+<junction x="2.54" y="91.44"/>
 </segment>
 </net>
@@
 <wire x1="81.28" y1="55.88" x2="81.28" y2="50.8" width="0.1524" layer="91"/>
 </segment>
+<segment>
+<pinref part="J2" gate="G$1" pin="GND"/>
+<pinref part="J3" gate="G$1" pin="GND"/>
+<wire x1="88.9" y1="106.68" x2="93.98" y2="106.68" width="0.1524" layer="91"/>
+<pinref part="GND3" gate="G$1" pin="GND"/>
+<wire x1="93.98" y1="106.68" x2="99.06" y2="106.68" width="0.1524" layer="91"/>
+<wire x1="93.98" y1="99.06" x2="93.98" y2="106.68" width="0.1524" layer="91"/>
+<junction x="93.98" y="106.68"/>
+</segment>
+<segment>
+<pinref part="J1" gate="G$1" pin="GND@6"/>
+<wire x1="7.62" y1="53.34" x2="2.54" y2="53.34" width="0.1524" layer="91"/>
+<wire x1="2.54" y1="53.34" x2="2.54" y2="50.8" width="0.1524" layer="91"/>
+<pinref part="J1" gate="G$1" pin="GND@9"/>
+<wire x1="2.54" y1="50.8" x2="2.54" y2="48.26" width="0.1524" layer="91"/>
+<wire x1="2.54" y1="48.26" x2="2.54" y2="45.72" width="0.1524" layer="91"/>
+<wire x1="2.54" y1="45.72" x2="2.54" y2="43.18" width="0.1524" layer="91"/>
+<wire x1="2.54" y1="43.18" x2="2.54" y2="40.64" width="0.1524" layer="91"/>
+<wire x1="2.54" y1="40.64" x2="2.54" y2="38.1" width="0.1524" layer="91"/>
+<wire x1="2.54" y1="38.1" x2="2.54" y2="35.56" width="0.1524" layer="91"/>
+<wire x1="2.54" y1="35.56" x2="2.54" y2="33.02" width="0.1524" layer="91"/>
+<wire x1="7.62" y1="50.8" x2="2.54" y2="50.8" width="0.1524" layer="91"/>
+<junction x="2.54" y="50.8"/>
+<pinref part="J1" gate="G$1" pin="GND@14"/>
+<wire x1="7.62" y1="48.26" x2="2.54" y2="48.26" width="0.1524" layer="91"/>
+<junction x="2.54" y="48.26"/>
+<pinref part="J1" gate="G$1" pin="GND@20"/>
+<wire x1="7.62" y1="45.72" x2="2.54" y2="45.72" width="0.1524" layer="91"/>
+<junction x="2.54" y="45.72"/>
+<pinref part="J1" gate="G$1" pin="GND@25"/>
+<wire x1="7.62" y1="43.18" x2="2.54" y2="43.18" width="0.1524" layer="91"/>
+<junction x="2.54" y="43.18"/>
+<pinref part="J1" gate="G$1" pin="GND@30"/>
+<wire x1="7.62" y1="40.64" x2="2.54" y2="40.64" width="0.1524" layer="91"/>
+<junction x="2.54" y="40.64"/>
+<pinref part="J1" gate="G$1" pin="GND@34"/>
+<wire x1="7.62" y1="38.1" x2="2.54" y2="38.1" width="0.1524" layer="91"/>
+<junction x="2.54" y="38.1"/>
+<pinref part="J1" gate="G$1" pin="GND@39"/>
+<wire x1="7.62" y1="35.56" x2="2.54" y2="35.56" width="0.1524" layer="91"/>
+<junction x="2.54" y="35.56"/>
+<pinref part="GND4" gate="G$1" pin="GND"/>
+</segment>
 </net>
 <net name="B" class="0">
@@
 <junction x="88.9" y="58.42"/>
 <label x="96.52" y="48.26" size="1.27" layer="95" xref="yes"/>
+</segment>
+<segment>
+<pinref part="J2" gate="G$1" pin="D-"/>
+<pinref part="J3" gate="G$1" pin="D-"/>
+<wire x1="88.9" y1="116.84" x2="96.52" y2="116.84" width="0.1524" layer="91"/>
+<wire x1="96.52" y1="116.84" x2="99.06" y2="116.84" width="0.1524" layer="91"/>
+<wire x1="96.52" y1="116.84" x2="96.52" y2="127" width="0.1524" layer="91"/>
+<wire x1="96.52" y1="127" x2="116.84" y2="127" width="0.1524" layer="91"/>
+<junction x="96.52" y="116.84"/>
+<label x="116.84" y="127" size="1.27" layer="95" xref="yes"/>
 </segment>
 </net>
@@
 <label x="96.52" y="68.58" size="1.27" layer="95" xref="yes"/>
 </segment>
+<segment>
+<pinref part="J2" gate="G$1" pin="D+"/>
+<pinref part="J3" gate="G$1" pin="D+"/>
+<wire x1="88.9" y1="111.76" x2="91.44" y2="111.76" width="0.1524" layer="91"/>
+<wire x1="91.44" y1="111.76" x2="99.06" y2="111.76" width="0.1524" layer="91"/>
+<wire x1="91.44" y1="111.76" x2="91.44" y2="132.08" width="0.1524" layer="91"/>
+<junction x="91.44" y="111.76"/>
+<wire x1="91.44" y1="132.08" x2="116.84" y2="132.08" width="0.1524" layer="91"/>
+<label x="116.84" y="132.08" size="1.27" layer="95" xref="yes"/>
+</segment>
 </net>

Commit message: first version for manufacturing
Parts:
- added J4: (no value), SparkFun-Connectors:CONN_05
- J3: value XLR-3-MALE -> (none); device SparkFun-Connectors:XLR-3-MALE -> SparkFun-Connectors:I2C_STANDARD
Connections:
- new net 3.3V: J1.3.3V@1, J1.3.3V@17, J3.2, J4.5
- new net DI: J1.GP5, U$1.DI
- new net MISO: J1.MISO, J4.3
- new net MOSI: J1.MOSI, J4.2
- new net SCL: J1.SCL, J3.4
- new net SCLK: J1.SCLK, J4.4
- new net SDA: J1.SDA, J3.3
- net 5V: now also U$1.DE
- net A: no longer J3.D+
- net B: no longer J3.D-
- net GND: now also J3.1, J4.1, U$1.RE, U$1.RO; no longer J3.GND
Other:
- moved on the sheet: R1, U$1
